Commit message: fix: rename karugamot2robot

File: robot_model/urdf/robot.urdf.xacro (robot description, xacro)
@@ -1,4 +1,4 @@
 <?xml version="1.0"?>
-<robot name="karugamot"
+<robot name="robot"
   xmlns:xacro="http://ros.org/wiki/xacro">
   <xacro:include filename="$(find robot_model)/urdf/common_properties.xacro"/>
@@ -11,5 +11,5 @@
       <origin xyz="0 0 -0.1" rpy="0 0 ${pi/2}"/>
       <geometry>
-        <mesh filename="package://robot_model/meshes/karugamot.stl" scale="0.001 0.001 0.001"/>
+        <mesh filename="package://robot_model/meshes/robot.stl" scale="0.001 0.001 0.001"/>
       </geometry>
       <material name="light_grey"/>
@@ -18,5 +18,5 @@
       <origin xyz="0 0 -0.1" rpy="0 0 ${pi/2}"/>
       <geometry>
-        <mesh filename="package://robot_model/meshes/karugamot.stl" scale="0.001 0.001 0.001"/>
+        <mesh filename="package://robot_model/meshes/robot.stl" scale="0.001 0.001 0.001"/>
       </geometry>
     </collision>
